Commit message: Added dvl_min_range and dvl_max_range to dvl params

File: uuv_sensor_plugins/uuv_sensor_ros_plugins/urdf/dvl_snippets.xacro (robot description, xacro)
@@ -66,5 +66,5 @@
     </xacro:dvl_plugin_macro>
   </xacro:macro>
-  <xacro:macro name="dvl_single_sonar" params="namespace suffix index pitch yaw update_rate">
+  <xacro:macro name="dvl_single_sonar" params="namespace suffix index pitch yaw update_rate dvl_min_range dvl_max_range">
     <link name="${namespace}/dvl${suffix}_sonar${index}_link">
       <inertial>
@@ -103,6 +103,6 @@
           </scan>
           <range>
-            <min>0.55</min>
-            <max>81</max>
+            <min>${dvl_min_range}</min>
+            <max>${dvl_max_range}</max>
             <resolution>0.01</resolution>
           </range>
@@ -122,5 +122,5 @@
   <xacro:macro name="dvl_plugin_macro"
     params="namespace suffix parent_link topic scale *origin update_rate
-    reference_frame noise_sigma noise_amplitude">
+    reference_frame noise_sigma noise_amplitude dvl_min_range dvl_max_range beam_angle">
     <link name="${namespace}/dvl${suffix}_link">
       <inertial>
@@ -145,17 +145,17 @@
     <xacro:dvl_single_sonar
       namespace="${namespace}" suffix=""
-      index="0" pitch="-0.52" yaw="0.0" update_rate="${update_rate}">
+      index="0" pitch="-${beam_angle}" yaw="0.0" update_rate="${update_rate}" dvl_min_range="${dvl_min_range}" dvl_max_range="${dvl_max_range}">
     </xacro:dvl_single_sonar>
     <xacro:dvl_single_sonar
       namespace="${namespace}" suffix=""
-      index="1" pitch="0" yaw="0.52" update_rate="${update_rate}">
+      index="1" pitch="0" yaw="${beam_angle}" update_rate="${update_rate}" dvl_min_range="${dvl_min_range}" dvl_max_range="${dvl_max_range}">
     </xacro:dvl_single_sonar>
     <xacro:dvl_single_sonar
       namespace="${namespace}" suffix=""
-      index="2" pitch="0.52" yaw="0.0" update_rate="${update_rate}">
+      index="2" pitch="${beam_angle}" yaw="0.0" update_rate="${update_rate}" dvl_min_range="${dvl_min_range}" dvl_max_range="${dvl_max_range}">
     </xacro:dvl_single_sonar>
     <xacro:dvl_single_sonar
       namespace="${namespace}" suffix=""
-      index="3" pitch="0.0" yaw="-0.52" update_rate="${update_rate}">
+      index="3" pitch="0.0" yaw="-${beam_angle}" update_rate="${update_rate}" dvl_min_range="${dvl_min_range}" dvl_max_range="${dvl_max_range}">
     </xacro:dvl_single_sonar>
     <gazebo>
